File: kicad/Gameboy-Interface-card/Gameboy-interface-card/Gameboy-interface-card.kicad_pcb (KiCad board)
At the start: 2 copper layers, 36 parts, among them J1 SCREEN, J2 RASPBERRY_PI, J3 BATERY, Q2 2N2222, SW1 BUTTON_A, SW2 BUTTON_B, SW3 BUTTON_SELECT, SW4 BUTTON_START, SW6 BUTTON_ARROW_DOWN, SW8 BUTTON_ARROW_RIGHT

Commit message: ok
Parts:
- moved G** 36.7 mm to (109.0, 131.5)
Routing:
- net SCREEN_CS: track 0.00 -> 209.0 mm, vias 0 -> 3
- net SCREEN_RESET: track 0.00 -> 173.3 mm, vias 0 -> 4
- net AUDIO: track 0.00 -> 116.9 mm, vias 0 -> 1
- net SELECT: track 50.9 -> 51.7 mm
Other:
- board outline added: 110.5 x 134 mm
